File: Project/Sporskiftecontroler/test1/test1.kicad_sch (KiCad schematic)
At the start: 0 parts

Commit message: mark subproject as dirty in history
Parts:
- added D1, D2: 1N5400, Diode_THT:D_DO-201AD_P15.24mm_Horizontal, symbol Diode:1N5400
- added D3: IR26-21C_L110_TR8, LED_SMD:LED_1206_3216Metric, symbol LED:IR26-21C_L110_TR8
- added J1: Conn_01x03_Pin, symbol Connector:Conn_01x03_Pin
- added J2, J3: Conn_01x02_Pin, symbol Connector:Conn_01x02_Pin
- added Q1: BC856, Package_TO_SOT_SMD:SOT-23, symbol Transistor_BJT:BC856
- added Q2: BC557, Package_TO_SOT_THT:TO-92_Inline, symbol Transistor_BJT:BC557
- added R1: R, symbol Device:R
- added U1: PC817, Package_DIP:DIP-4_W7.62mm, symbol Isolator:PC817
Connections:
- new net: J1.3 (Pin_3), R1.1
- new net: J2.2 (Pin_2), J3.2 (Pin_2), R1.2, U1.2
- new net: D3.1 (K), J2.1 (Pin_1), J3.1 (Pin_1), U1.1
- new net: D1.2 (A), D2.1 (K), J1.1 (Pin_1), Q1.2 (E)
- new net: D1.1 (K), D2.2 (A), J1.2 (Pin_2), Q1.1 (B)
- new net: D3.2 (A), Q1.3 (C)
Other:
- note added: "DCC GND"
- note added: "DCC Power"
- note added: "DCC Track"
