File: Project/BlockDetection/Moppe/Moppe.kicad_sch (KiCad schematic)
At the start: 12 parts, among them J1 Conn_01x03_Pin, J2 Conn_01x02_Pin, J3 Conn_01x02_Pin, Q1 BC856 or BC557, U1 PC817

Commit message: SporBesat a la´ Moppe
Parts:
- removed C2: 100nF, symbol Device:C
- removed J2, J3: Conn_01x02_Pin, symbol Connector:Conn_01x02_Pin
Connections:
- net at Q1.3 (C), R1.2: no longer C1.2
- net at D3.1 (K), U1.1: now also C1.1
- net at J1.3 (Pin_3), U1.2: now also C1.2
- net at D1.2 (A), D2.1 (K), J1.1 (Pin_1)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: no longer C1.1
Other:
- moved on the sheet: C1, R2, U1

Commit message: SporBesat a la´ Moppe
Parts:
- added J2: Conn_01x02_Pin, Connector:Tag-Connect_TC2030-IDC-FP_2x03_P1.27mm_Vertical, symbol Connector:Conn_01x02_Pin
Connections:
- net at U1.3: now also J2.1 (Pin_1)
- net at U1.4: now also J2.2 (Pin_2)
Changed lines of the file:
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@@
+	(wire
+		(pts
+			(xy 143.51 111.76) (xy 153.67 111.76)
+		)
+		(stroke
+			(width 0)
+			(type default)
+		)
+	)
 	(wire
 		(pts
@@
 	(wire
 		(pts
+			(xy 147.32 106.68) (xy 147.32 109.22)
+		)
+		(stroke
+			(width 0)
+			(type default)
+		)
+	)
+	(wire
+		(pts
 			(xy 86.36 69.85) (xy 86.36 72.39)
 		)
@@
 	(wire
 		(pts
+			(xy 143.51 106.68) (xy 147.32 106.68)
+		)
+		(stroke
+			(width 0)
+			(type default)
+		)
+	)
+	(wire
+		(pts
 			(xy 74.93 64.77) (xy 78.74 64.77)
 		)
@@
 			(width 0)
 			(type default)
+		)
+	)
+	(wire
+		(pts
+			(xy 147.32 109.22) (xy 153.67 109.22)
+		)
+		(stroke
+			(width 0)
+			(type default)
+		)
+	)
+	(label "MCU Input"
+		(at 160.02 110.49 0)
+		(effects
+			(font
+				(size 1.27 1.27)
+			)
+			(justify left bottom)
+		)
+	)
+	(label "MCU Gnd"
+		(at 160.02 113.03 0)
+		(effects
+			(font
+				(size 1.27 1.27)
+			)
+			(justify left bottom)
 		)
 	)
@@
 					(unit 1)
 				)
+			)
+		)
+	)
+	(symbol
+		(lib_id "Connector:Conn_01x02_Pin")
+		(at 158.75 111.76 180)
+		(unit 1)
+		(body_style 1)
+		(exclude_from_sim no)
+		(in_bom yes)
+		(on_board yes)
+		(in_pos_files yes)
+		(dnp no)
+		(property "Reference" "J2"
+			(at 154.686 105.156 0)
+			(show_name no)
+			(do_not_autoplace no)
+			(effects
+				(font
+					(size 1.27 1.27)
+				)
+				(justify right)
+			)
+		)
+		(property "Value" "Conn_01x02_Pin"
+			(at 160.274 104.394 0)
+			(hide yes)
+			(show_name no)
+			(do_not_autoplace no)
+			(effects
+				(font
+					(size 1.27 1.27)
+				)
+				(justify right)
+			)
+		)
+		(property "Footprint" "Connector:Tag-Connect_TC2030-IDC-FP_2x03_P1.27mm_Vertical"
+			(at 158.75 111.76 0)
+			(hide yes)
+			(show_name no)
+			(do_not_autoplace no)
+			(effects
+				(font
+					(size 1.27 1.27)
+				)
+			)
+		)
+		(property "Datasheet" ""
+			(at 158.75 111.76 0)
+			(hide yes)
+			(show_name no)
+			(do_not_autoplace no)
+			(effects
+				(font
+					(size 1.27 1.27)
+				)
+			)
+		)
+		(property "Description" "Generic connector, single row, 01x02, script generated"
+			(at 158.75 111.76 0)
+			(hide yes)
+			(show_name no)
+			(do_not_autoplace no)
+			(effects
+				(font
+					(size 1.27 1.27)
+				)
+			)
+		)
+		(pin "1"
+		)
+		(pin "2"
+		)
+		(instances
+			(project "Moppe"
+				(path "/df40a3ed-29e1-4fed-8bb8-557e0f8da153"
+					(reference "J2")
+					(unit 1)
+				)

Commit message: SporBesat a la´ Moppe
Parts:
- removed J1: Conn_01x03_Pin, symbol Connector:Conn_01x03_Pin
- added J1, J2, J3: Conn_01x02_Pin, Connector:Tag-Connect_TC2030-IDC-FP_2x03_P1.27mm_Vertical, symbol Connector:Conn_01x02_Pin
Connections:
- net at C1.2, U1.2: now also J1.1 (Pin_1), J2.1 (Pin_1), J3.1 (Pin_1)
- net at D1.2 (A), D2.1 (K), Q1.2 (E): now also J1.2 (Pin_2), J2.2 (Pin_2)
- net at D1.1 (K), D2.2 (A), R2.2: now also J3.2 (Pin_2)
Other:
- note removed: "DCC GND"
- note removed: "DCC Power"
- note removed: "DCC Track"
- moved on the sheet: C1, D3, J2, Q1, R1, R2, U1

Commit message: SporBesat a la´ Moppe
Parts:
- added C2, C3, C4: 10 µF, symbol Device:C_Polarized_Small
- added D10, D4, D7: 1N5400 or S5AC, Diode_THT:D_DO-201AD_P15.24mm_Horizontal, symbol Diode:1N5400
- added D11, D5, D8: 1N5400, Diode_THT:D_DO-201AD_P15.24mm_Horizontal, symbol Diode:1N5400
- added D12, D6, D9: IR26-21C_L110_TR8, LED_SMD:LED_1206_3216Metric, symbol LED:IR26-21C_L110_TR8
- added J11, J12, J13, J4, J5, J6: Conn_01x02_Pin, Connector:Tag-Connect_TC2030-IDC-FP_2x03_P1.27mm_Vertical, symbol Connector:Conn_01x02_Pin
- added Q2, Q3, Q4: BC856 or BC557, Package_TO_SOT_SMD:SOT-23, symbol Transistor_BJT:BC856
- added R3, R5, R7: 10R, symbol Device:R
- added R4, R6, R8: 1K8, symbol Device:R
- added U2, U3, U4: PC817, Package_DIP:DIP-4_W7.62mm, symbol Isolator:PC817
- renumbered J2 to J10
Connections:
- net at C1.2, J1.1 (Pin_1), J2.1 (Pin_1)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: now also C2.2, C3.2, C4.2, J4.1 (Pin_1), J5.1 (Pin_1), J6.1 (Pin_1), U2.2, U3.2, U4.2
- net at D1.2 (A), D2.1 (K), J1.2 (Pin_2)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: now also D10.2 (A), D11.1 (K), D4.2 (A), D5.1 (K), D7.2 (A), D8.1 (K), Q2.2 (E), Q3.2 (E), Q4.2 (E)
- new net: D4.1 (K), D5.2 (A), J4.2 (Pin_2), R3.2
- new net: C4.1, D12.1 (K), U4.1
- new net: J12.1 (Pin_1), U3.3
- new net: J12.2 (Pin_2), U3.4
- new net: D6.2 (A), R4.1
- new net: Q2.3 (C), R4.2
- new net: Q2.1 (B), R3.1
- new net: C2.1, D6.1 (K), U2.1
- new net: D7.1 (K), D8.2 (A), J5.2 (Pin_2), R5.2
- new net: D9.2 (A), R6.1
- new net: Q3.3 (C), R6.2
- new net: J11.1 (Pin_1), U2.3
- new net: J11.2 (Pin_2), U2.4
- new net: D12.2 (A), R8.1
- new net: C3.1, D9.1 (K), U3.1
- new net: Q3.1 (B), R5.1
- new net: Q4.1 (B), R7.1
- new net: D10.1 (K), D11.2 (A), J6.2 (Pin_2), R7.2
- new net: Q4.3 (C), R8.2
- new net: J13.1 (Pin_1), U4.3
- new net: J13.2 (Pin_2), U4.4
Other:
- moved on the sheet: C1, D1, D2, D3, J1, J10, J2, J3, Q1, R1, R2, U1

Commit message: SporBesat a la´ Moppe
Parts:
- removed J10, J11, J12, J13: Conn_01x02_Pin, Connector:Tag-Connect_TC2030-IDC-FP_2x03_P1.27mm_Vertical, symbol Connector:Conn_01x02_Pin
- removed U1, U2, U3, U4: PC817, Package_DIP:DIP-4_W7.62mm, symbol Isolator:PC817
- added J7: RJ45_Shielded, Connector_RJ:RJ45_Bel_V895-1001-AW_Vertical, symbol Connector:RJ45_Shielded
- added U5: PC847, Package_DIP:DIP-16_W7.62mm, symbol Isolator:PC847
Connections:
- net at C4.1, D12.1 (K): now also U5.7
- net at C1.2, C2.2, C3.2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: now also U5.2, U5.4, U5.6, U5.8
- net at C1.1, D3.1 (K): now also U5.1
- net at C2.1, D6.1 (K): now also U5.3
- net at C3.1, D9.1 (K): now also U5.5
- new net: J7.2, U5.15
- new net: J7.1, U5.16
- new net: J7.4, U5.11
- new net: J7.5, U5.12
- new net: J7.6, U5.13
- new net: J7.3, U5.14
- new net: J7.7, U5.10
- new net: J7.8, U5.9

Commit message: Anotade
Parts:
- D1: value 1N5400 or S5AC -> S5AC
- J7: value RJ45_Shielded -> Amphenol RJHSE5380; footprint Connector_RJ:RJ45_Bel_V895-1001-AW_Vertical -> Connector_RJ:RJ45_Amphenol_RJHSE5380
- Q1: value BC856 or BC557 -> BC856
- renumbered D6 to D10, D9 to D11, D4 to D2, D7 to D3, D10 to D4, D2 to D5, D5 to D6, D8 to D7, D11 to D8, D3 to D9, R2 to R1, R3 to R2, R5 to R3, R7 to R4, R1 to R5, R4 to R6, R6 to R7, U5 to U1

Commit message: moppe
Parts:
- added D13: D_Bridge_+-AA, Module:Pololu_Breakout-16_15.2x20.3mm, symbol Device:D_Bridge_+-AA
- added R10: 22R, symbol Device:R
- added R9: 470R, symbol Device:R
- added U2: PC817, Package_DIP:DIP-4_W7.62mm, symbol Isolator:PC817
Connections:
- net at C1.2, C2.2, C3.2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: now also D13.4, R9.2, U2.2
- net at D1.2 (A), D2.2 (A), D3.2 (A)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: now also D13.3, R10.2, R9.1
- new net: D13.1 (+), D13.2 (-)
- new net: R10.1, U2.1

Commit message: moppe bro
Parts:
- added J8: Conn_01x02_Pin, Connector:Tag-Connect_TC2030-IDC-FP_2x03_P1.27mm_Vertical, symbol Connector:Conn_01x02_Pin
Connections:
- net at C1.2, C2.2, C3.2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: now also J8.1 (Pin_1); no longer D13.4, R9.2, U2.2
- new net: D13.4, J8.2 (Pin_2), R9.2, U2.2
